Commit message: added collision factors manually

File: urdf/atcart_greenhouse_gazebo.urdf (robot description, URDF)
Before this commit: robot atcart_greenhouse_gazebo, 9 links, 8 joints
Links:
- link base_link: geometry collision box size=0.48 0.26 0.18; visual mesh filename=package://atcart_greenhouse_gazebo/meshes/base_link.STL
- link caster_holder_left: geometry collision cylinder length=0.025 radius=0.03; visual mesh filename=package://atcart_greenhouse_gazebo/meshes/caster_holder_lef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
- link caster_holder_right: geometry collision cylinder length=0.025 radius=0.03; visual mesh filename=package://atcart_greenhouse_gazebo/meshes/caster_holder_rig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
- link caster_wheel_left: geometry collision cylinder length=0.04 radius=0.051; visual mesh filename=package://atcart_greenhouse_gazebo/meshes/caster_wheel_left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
- link caster_wheel_right: geometry collision cylinder length=0.04 radius=0.051; visual mesh filename=package://atcart_greenhouse_gazebo/meshes/caster_wheel_righ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
- link rear_wheel_left: geometry collision cylinder length=0.1143 radius=0.16; visual mesh filename=package://atcart_greenhouse_gazebo/meshes/rear_wheel_left.S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
- link rear_wheel_right: geometry collision cylinder length=0.1143 radius=0.16; visual mesh filename=package://atcart_greenhouse_gazebo/meshes/rear_wheel_right.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
