Commit message: changed file name

File: urdf/atcart_basic_gazebo.urdf (robot description, URDF)
Before this commit: robot atcart_greenhouse_gazebo, 9 links, 8 joints
Links:
- link base_link: geometry collision box size=0.48 0.26 0.18; visual mesh filename=package://atcart_basic_gazebo/meshes/base_link.STL
- link caster_holder_left: geometry collision cylinder length=0.025 radius=0.03; visual mesh filename=package://atcart_basic_gazebo/meshes/caster_holder_left.STL
- link caster_holder_right: geometry collision cylinder length=0.025 radius=0.03; visual mesh filename=package://atcart_basic_gazebo/meshes/caster_holder_right.STL
- link caster_wheel_left: geometry collision cylinder length=0.04 radius=0.051; visual mesh filename=package://atcart_basic_gazebo/meshes/caster_wheel_left.STL
- link caster_wheel_right: geometry collision cylinder length=0.04 radius=0.051; visual mesh filename=package://atcart_basic_gazebo/meshes/caster_wheel_right.STL
- link rear_wheel_left: geometry collision cylinder length=0.1143 radius=0.16; visual mesh filename=package://atcart_basic_gazebo/meshes/rear_wheel_left.STL
- link rear_wheel_right: geometry collision cylinder length=0.1143 radius=0.16; visual mesh filename=package://atcart_basic_gazebo/meshes/rear_wheel_right.STL
